Commit message: astra position, sensor poles, robot.model.xml
Fix astra position, fixes #1
Xacro for sensor_poles, kinect_poles, astra_poles in hexagons.urdf.xacro
  Change or remove sensor poles from turtlebot
Launch files formatted to pass params to launch/includes/robot.model.xml

File: robots/kobuki_hexagons_astra_.8m_tall.urdf.xacro (robot description, xacro)
@@ -8,10 +8,10 @@
   <xacro:include filename="$(find turtlebot_description)/urdf/turtlebot_common_library.urdf.xacro" />
   <xacro:include filename="$(find kobuki_description)/urdf/kobuki.urdf.xacro" />
-  <xacro:include filename="$(find turtlebot_description)/urdf/stacks/hexagons.urdf.xacro"/>
+  <xacro:include filename="$(find turtlebot_custom_description)/urdf/stacks/hexagons.urdf.xacro"/>
   <xacro:include filename="$(find turtlebot_custom_description)/urdf/stacks/extended_top_1m.urdf.xacro"/>
   <xacro:include filename="$(find turtlebot_custom_description)/urdf/sensors/astra.urdf.xacro"/>
   <xacro:include filename="$(find turtlebot_custom_description)/urdf/sensors/razor_9dof_m0.urdf.xacro"/>
   <kobuki/>
-  <stack_hexagons parent="base_link"/>
+  <stack_hexagons parent="base_link" sensor_poles="false"/>
   <stack_extended_top_1m parent="base_link"/>
   <sensor_astra parent="base_link" cam_pz="1.30635"/>

File: urdf/sensors/astra.urdf.xacro (robot description, xacro)
@@ -41,6 +41,6 @@
     <link name="camera_rgb_optical_frame"/>
     <joint name="camera_joint" type="fixed">
-      <origin xyz="0 ${astra_cam_rel_rgb_py} 0"
-              rpy="0 0 0"/>
+      <origin xyz="-0.0075 0 0"
+              rpy="0 0 0"/><!-- 0 ${astra_cam_rel_rgb_py} 0 -->
       <parent link="camera_rgb_frame"/>
       <child link="camera_link"/>
@@ -48,5 +48,5 @@
     <link name="camera_link">
       <visual>
-        <origin xyz="0 .021 0" rpy="0 0 ${M_PI/2}"/>
+        <origin xyz="0 0 0" rpy="0 0 ${M_PI/2}"/> <!-- 0 0.021 0 -->
         <geometry>
           <mesh filename="package://turtlebot_custom_description/meshes/sensors/astra.STL" scale="${astra_dae_display_scale} ${astra_dae_display_scale} ${astra_dae_display_scale}"/>
